Commit message: description: v119 model with housing, Gemini 2 camera and 18 kg mass
URDF/Xacro and meshes from AMR_MASTER_Linear v119 (see
src/amr_description/reports/UPDATE_V119.md): four-piece housing
(X +-328, Y +-278 mm, fenders to Z 100 mm), Orbbec Gemini 2 in the
housing nose pitched 12 deg up, rear XT90 connector. camera_link sits on
the left IR lens axis; OrbbecSDK_ROS2 publishes the frames below it. The
housing and fender boxes replace the lower-frame and suspension colliders.
The STEP stays out of git (hash in input_sha256.json).

The housing makes the body 0.656 m long: the local costmap footprint and
the RL scan footprint become X +-0.328 m. Total mass is set to 18.0 kg,
the 3.0 kg increase on base_link; the physics URDF check and the Isaac
runtime check now expect 18 kg.

Isaac Sim: re-imported; runtime test, passive, floor4 stability and floor
contact checks pass, and six full-stack scenarios reach the goal without
contact.

Co-Authored-By: Claude Opus 5.5 <noreply@anthropic.com>

File: src/amr_description/urdf/capstone_amr.urdf (robot description, URDF)
Before this commit: robot capstone_amr, 20 links, 19 joints
Links:
- added link camera_link
- link base_link: mass 9.8 -> 12.8; geometry collision box size=0.010 0.060 0.050; collision box size=0.010 0.060 0.050
Joints:
- added joint camera_joint: type fixed, parent base_link, child camera_link, origin xyz=0.320488 0.025 0.061017 rpy=0 -0.20943951023931953 0

File: src/amr_description/urdf/capstone_amr.urdf.xacro (robot description, xacro)
@@ -8,6 +8,8 @@
     Geometry revision: AMR_MASTER_Linear v80.step (2026-10-16): aluminium
     profile frame with upper structure, Z10T mast, linear-guide drive-wheel
-    suspension (modelled rigid) and 529 mm drive track. The v28 measured mass
-    budget and base_link inertia approximation are retained until reweighed.
+    suspension (modelled rigid) and 529 mm drive track. The base_link inertia
+    box approximation from v28 is retained.
+    v119 (2026-10-20) adds the four-piece housing, an Orbbec Gemini 2 depth
+    camera in the housing nose (pitched 12 deg up) and the rear XT90 connector.
     Direct Isaac Sim import uses the expanded capstone_amr.urdf beside this file.
     Import as Robot Type=Wheeled, Base Type=Mobile, with self-collision disabled.
@@ -21,21 +23,36 @@
   <xacro:property name="drive_wheel_mesh_scale" value="0.001004086"/>
   <xacro:property name="drive_wheel_mesh_y" value="0.029118494"/>
-  <!-- v28 base_link inertia box, retained until the v80 robot is reweighed. -->
+  <!-- v28 base_link inertia box, retained until the robot is reweighed. -->
   <xacro:property name="base_inertia_length" value="0.640"/>
   <xacro:property name="base_inertia_width" value="0.520"/>
   <xacro:property name="base_inertia_height" value="0.085"/>
   <xacro:property name="base_inertia_center_z" value="-0.0115"/>
-  <!-- v80 lower profile frame: X +-320, Y +-260, Z -54 to 1 mm. -->
-  <xacro:property name="frame_length" value="0.640"/>
-  <xacro:property name="frame_width" value="0.520"/>
-  <xacro:property name="frame_bottom_z" value="-0.054"/>
-  <xacro:property name="frame_top_z" value="0.001"/>
-  <!--
-    15.0 kg measured total mass budget:
-      base_link remainder 9.8 kg (battery, frame, plate, electronics, LiDAR and mount)
-      two drive wheels 2 x 2.2 kg, four complete casters 4 x 0.2 kg.
+  <!--
+    v119 housing outer bounds: X +-328, Y +-278, Z -55 to 80 mm, with fenders
+    over the drive wheels (X +-114, |Y| 180 to 278 mm) up to Z 100 mm. It
+    encloses the lower profile frame (X +-320, Y +-260, Z -54 to 1 mm).
+  -->
+  <xacro:property name="housing_length" value="0.656"/>
+  <xacro:property name="housing_width" value="0.556"/>
+  <xacro:property name="housing_bottom_z" value="-0.055"/>
+  <xacro:property name="housing_top_z" value="0.080"/>
+  <!--
+    Gemini 2 in the v119 STEP: body origin at base_link (311, 0, 59) mm, optical
+    axes pitched 12 deg up. camera_link is the left (+Y) IR lens front on its
+    optical axis, where the Orbbec driver's depth frame is assumed to sit.
+  -->
+  <xacro:property name="camera_x" value="0.320488"/>
+  <xacro:property name="camera_y" value="0.025"/>
+  <xacro:property name="camera_z" value="0.061017"/>
+  <xacro:property name="camera_pitch" value="${-12.0 * pi / 180.0}"/>
+  <!--
+    18.0 kg total mass (set 2026-10-20 for v119; v28 measured 15.0 kg):
+      base_link remainder 12.8 kg (battery, frame, upper frame, mast, Z10T,
+        housing, electronics, LiDAR, Gemini 2 and their mounts)
+      two drive wheels 2 x 2.2 kg, four complete casters 4 x 0.2 kg (measured).
     Each caster's measured 0.2 kg is provisionally split across its three links.
-  -->
-  <xacro:property name="chassis_mass" value="9.8"/>
+    The 3.0 kg increase is all on base_link, inside the v28 inertia box below.
+  -->
+  <xacro:property name="chassis_mass" value="12.8"/>
   <xacro:property name="drive_wheel_mass" value="2.2"/>
   <xacro:property name="caster_mount_mass" value="0.05"/>
@@ -54,4 +71,7 @@
     <color rgba="0.12 0.13 0.15 1"/>
   </material>
+  <material name="housing">
+    <color rgba="0.82 0.83 0.84 1"/>
+  </material>
   <material name="rubber">
     <color rgba="0.04 0.045 0.055 1"/>
@@ -89,5 +109,6 @@
       x="${base_inertia_length}" y="${base_inertia_width}" z="${base_inertia_height}"
       origin_xyz="0 0 ${base_inertia_center_z}"/>
-    <!-- These three STLs are already expressed in the base_link CAD frame. -->
+    <!-- These four STLs are already expressed in the base_link CAD frame.
+         chassis.stl also carries the rear XT90 connector. -->
     <visual>
       <origin xyz="0 0 0" rpy="0 0 0"/>
@@ -112,4 +133,20 @@
       <material name="z10t_body"/>
     </visual>
+    <visual>
+      <origin xyz="0 0 0" rpy="0 0 0"/>
+      <geometry>
+        <mesh filename="${mesh_prefix}/housing.stl" scale="0.001 0.001 0.001"/>
+      </geometry>
+      <material name="housing"/>
+    </visual>
+    <!-- Camera geometry is lumped into base_link like the LiDAR;
+         gemini2.stl is expressed in the camera_link frame. -->
+    <visual>
+      <origin xyz="${camera_x} ${camera_y} ${camera_z}" rpy="0 ${camera_pitch} 0"/>
+      <geometry>
+        <mesh filename="${mesh_prefix}/gemini2.stl" scale="0.001 0.001 0.001"/>
+      </geometry>
+      <material name="z10t_body"/>
+    </visual>
     <!-- LiDAR geometry is lumped into base_link together with its mass. -->
     <visual>
@@ -127,12 +164,16 @@
       <material name="dark_metal"/>
     </visual>
-    <!-- PhysX-friendly collision boxes from the v80 part bounds; the visual
-         frame STL has 287,840 triangles. -->
-    <collision>
-      <origin xyz="0 0 ${(frame_bottom_z + frame_top_z) / 2.0}" rpy="0 0 0"/>
-      <geometry>
-        <box size="${frame_length} ${frame_width} ${frame_top_z - frame_bottom_z}"/>
-      </geometry>
-    </collision>
+    <!-- PhysX-friendly collision boxes from the v119 part bounds. The housing
+         box also covers the lower frame, the suspension brackets, the camera
+         (front at X 324 mm) and the XT90 connector (rear at X -326 mm). -->
+    <collision>
+      <origin xyz="0 0 ${(housing_bottom_z + housing_top_z) / 2.0}" rpy="0 0 0"/>
+      <geometry>
+        <box size="${housing_length} ${housing_width} ${housing_top_z - housing_bottom_z}"/>
+      </geometry>
+    </collision>
+    <!-- Fenders over the drive wheels. -->
+    <xacro:frame_box x="0" y="0.229" z="0.090" sx="0.228" sy="0.098" sz="0.020"/>
+    <xacro:frame_box x="0" y="-0.229" z="0.090" sx="0.228" sy="0.098" sz="0.020"/>
     <!-- 2020 uprights. They cross the LiDAR scan plane at Z = 108.605 mm. -->
     <xacro:frame_box x="0.270" y="0.1326" z="0.066" sx="0.020" sy="0.040" sz="0.200"/>
@@ -148,7 +189,4 @@
     <xacro:frame_box x="0.2372" y="0" z="0.6035" sx="0.0764" sy="0.100" sz="0.055"/>
     <xacro:frame_box x="0.2308" y="0" z="0.6925" sx="0.123" sy="0.233" sz="0.123"/>
-    <!-- Drive-wheel suspension brackets above the lower frame. -->
-    <xacro:frame_box x="0" y="0.2075" z="0.013" sx="0.200" sy="0.055" sz="0.094"/>
-    <xacro:frame_box x="0" y="-0.2075" z="0.013" sx="0.200" sy="0.055" sz="0.094"/>
     <!-- v3 mount: two extended walls, two upper side walls, and top plate.
          Small counterbored screw holes are omitted from collision geometry. -->
@@ -305,3 +343,15 @@
     <origin xyz="0.160 0.0035 0.016" rpy="0 0 0"/>
   </joint>
+  <!--
+    Orbbec Gemini 2 mount frame (+X along the optical axis, +Z up, pitched
+    12 deg up). OrbbecSDK_ROS2 publishes camera_link -> depth/color/IR and
+    optical frames itself from the factory calibration, so none of those
+    frames are defined here. Depth FOV 91 x 66 deg, 50 mm baseline.
+  -->
+  <link name="camera_link"/>
+  <joint name="camera_joint" type="fixed">
+    <parent link="base_link"/>
+    <child link="camera_link"/>
+    <origin xyz="${camera_x} ${camera_y} ${camera_z}" rpy="0 ${camera_pitch} 0"/>
+  </joint>
 </robot>

File: src/amr_description/urdf/capstone_amr_physics.urdf (robot description, URDF)
Before this commit: robot capstone_amr, 20 links, 19 joints
Links:
- added link camera_link
- link base_link: mass 9.8 -> 12.8; geometry collision box size=0.010 0.060 0.050; collision box size=0.010 0.060 0.050
Joints:
- added joint camera_joint: type fixed, parent base_link, child camera_link, origin xyz=0.320488 0.025 0.061017 rpy=0 -0.20943951023931953 0

File: src/amr_description/urdf/capstone_amr_physics.urdf.xacro (robot description, xacro)
@@ -9,6 +9,8 @@
     Geometry revision: AMR_MASTER_Linear v80.step (2026-10-16): aluminium
     profile frame with upper structure, Z10T mast, linear-guide drive-wheel
-    suspension (modelled rigid) and 529 mm drive track. The v28 measured mass
-    budget and base_link inertia approximation are retained until reweighed.
+    suspension (modelled rigid) and 529 mm drive track. The base_link inertia
+    box approximation from v28 is retained.
+    v119 (2026-10-20) adds the four-piece housing, an Orbbec Gemini 2 depth
+    camera in the housing nose (pitched 12 deg up) and the rear XT90 connector.
     Direct Isaac Sim import uses the expanded capstone_amr.urdf beside this file.
     Import as Robot Type=Wheeled, Base Type=Mobile, with self-collision disabled.
@@ -22,21 +24,36 @@
   <xacro:property name="drive_wheel_mesh_scale" value="0.001004086"/>
   <xacro:property name="drive_wheel_mesh_y" value="0.029118494"/>
-  <!-- v28 base_link inertia box, retained until the v80 robot is reweighed. -->
+  <!-- v28 base_link inertia box, retained until the robot is reweighed. -->
   <xacro:property name="base_inertia_length" value="0.640"/>
   <xacro:property name="base_inertia_width" value="0.520"/>
   <xacro:property name="base_inertia_height" value="0.085"/>
   <xacro:property name="base_inertia_center_z" value="-0.0115"/>
-  <!-- v80 lower profile frame: X +-320, Y +-260, Z -54 to 1 mm. -->
-  <xacro:property name="frame_length" value="0.640"/>
-  <xacro:property name="frame_width" value="0.520"/>
-  <xacro:property name="frame_bottom_z" value="-0.054"/>
-  <xacro:property name="frame_top_z" value="0.001"/>
-  <!--
-    15.0 kg measured total mass budget:
-      base_link remainder 9.8 kg (battery, frame, plate, electronics, LiDAR and mount)
-      two drive wheels 2 x 2.2 kg, four complete casters 4 x 0.2 kg.
+  <!--
+    v119 housing outer bounds: X +-328, Y +-278, Z -55 to 80 mm, with fenders
+    over the drive wheels (X +-114, |Y| 180 to 278 mm) up to Z 100 mm. It
+    encloses the lower profile frame (X +-320, Y +-260, Z -54 to 1 mm).
+  -->
+  <xacro:property name="housing_length" value="0.656"/>
+  <xacro:property name="housing_width" value="0.556"/>
+  <xacro:property name="housing_bottom_z" value="-0.055"/>
+  <xacro:property name="housing_top_z" value="0.080"/>
+  <!--
+    Gemini 2 in the v119 STEP: body origin at base_link (311, 0, 59) mm, optical
+    axes pitched 12 deg up. camera_link is the left (+Y) IR lens front on its
+    optical axis, where the Orbbec driver's depth frame is assumed to sit.
+  -->
+  <xacro:property name="camera_x" value="0.320488"/>
+  <xacro:property name="camera_y" value="0.025"/>
+  <xacro:property name="camera_z" value="0.061017"/>
+  <xacro:property name="camera_pitch" value="${-12.0 * pi / 180.0}"/>
+  <!--
+    18.0 kg total mass (set 2026-10-20 for v119; v28 measured 15.0 kg):
+      base_link remainder 12.8 kg (battery, frame, upper frame, mast, Z10T,
+        housing, electronics, LiDAR, Gemini 2 and their mounts)
+      two drive wheels 2 x 2.2 kg, four complete casters 4 x 0.2 kg (measured).
     Each caster's measured 0.2 kg is provisionally split across its three links.
-  -->
-  <xacro:property name="chassis_mass" value="9.8"/>
+    The 3.0 kg increase is all on base_link, inside the v28 inertia box below.
+  -->
+  <xacro:property name="chassis_mass" value="12.8"/>
   <xacro:property name="drive_wheel_mass" value="2.2"/>
   <xacro:property name="caster_mount_mass" value="0.05"/>
@@ -55,4 +72,7 @@
     <color rgba="0.12 0.13 0.15 1"/>
   </material>
+  <material name="housing">
+    <color rgba="0.82 0.83 0.84 1"/>
+  </material>
   <material name="rubber">
     <color rgba="0.04 0.045 0.055 1"/>
@@ -90,5 +110,6 @@
       x="${base_inertia_length}" y="${base_inertia_width}" z="${base_inertia_height}"
       origin_xyz="0 0 ${base_inertia_center_z}"/>
-    <!-- These three STLs are already expressed in the base_link CAD frame. -->
+    <!-- These four STLs are already expressed in the base_link CAD frame.
+         chassis.stl also carries the rear XT90 connector. -->
     <visual>
       <origin xyz="0 0 0" rpy="0 0 0"/>
@@ -113,4 +134,20 @@
       <material name="z10t_body"/>
     </visual>
+    <visual>
+      <origin xyz="0 0 0" rpy="0 0 0"/>
+      <geometry>
+        <mesh filename="${mesh_prefix}/housing.stl" scale="0.001 0.001 0.001"/>
+      </geometry>
+      <material name="housing"/>
+    </visual>
+    <!-- Camera geometry is lumped into base_link like the LiDAR;
+         gemini2.stl is expressed in the camera_link frame. -->
+    <visual>
+      <origin xyz="${camera_x} ${camera_y} ${camera_z}" rpy="0 ${camera_pitch} 0"/>
+      <geometry>
+        <mesh filename="${mesh_prefix}/gemini2.stl" scale="0.001 0.001 0.001"/>
+      </geometry>
+      <material name="z10t_body"/>
+    </visual>
     <!-- LiDAR geometry is lumped into base_link together with its mass. -->
     <visual>
@@ -128,12 +165,16 @@
       <material name="dark_metal"/>
     </visual>
-    <!-- PhysX-friendly collision boxes from the v80 part bounds; the visual
-         frame STL has 287,840 triangles. -->
-    <collision>
-      <origin xyz="0 0 ${(frame_bottom_z + frame_top_z) / 2.0}" rpy="0 0 0"/>
-      <geometry>
-        <box size="${frame_length} ${frame_width} ${frame_top_z - frame_bottom_z}"/>
-      </geometry>
-    </collision>
+    <!-- PhysX-friendly collision boxes from the v119 part bounds. The housing
+         box also covers the lower frame, the suspension brackets, the camera
+         (front at X 324 mm) and the XT90 connector (rear at X -326 mm). -->
+    <collision>
+      <origin xyz="0 0 ${(housing_bottom_z + housing_top_z) / 2.0}" rpy="0 0 0"/>
+      <geometry>
+        <box size="${housing_length} ${housing_width} ${housing_top_z - housing_bottom_z}"/>
+      </geometry>
+    </collision>
+    <!-- Fenders over the drive wheels. -->
+    <xacro:frame_box x="0" y="0.229" z="0.090" sx="0.228" sy="0.098" sz="0.020"/>
+    <xacro:frame_box x="0" y="-0.229" z="0.090" sx="0.228" sy="0.098" sz="0.020"/>
     <!-- 2020 uprights. They cross the LiDAR scan plane at Z = 108.605 mm. -->
     <xacro:frame_box x="0.270" y="0.1326" z="0.066" sx="0.020" sy="0.040" sz="0.200"/>
@@ -149,7 +190,4 @@
     <xacro:frame_box x="0.2372" y="0" z="0.6035" sx="0.0764" sy="0.100" sz="0.055"/>
     <xacro:frame_box x="0.2308" y="0" z="0.6925" sx="0.123" sy="0.233" sz="0.123"/>
-    <!-- Drive-wheel suspension brackets above the lower frame. -->
-    <xacro:frame_box x="0" y="0.2075" z="0.013" sx="0.200" sy="0.055" sz="0.094"/>
-    <xacro:frame_box x="0" y="-0.2075" z="0.013" sx="0.200" sy="0.055" sz="0.094"/>
     <!-- v3 mount: two extended walls, two upper side walls, and top plate.
          Small counterbored screw holes are omitted from collision geometry. -->
@@ -307,3 +345,15 @@
     <origin xyz="0.160 0.0035 0.016" rpy="0 0 0"/>
   </joint>
+  <!--
+    Orbbec Gemini 2 mount frame (+X along the optical axis, +Z up, pitched
+    12 deg up). OrbbecSDK_ROS2 publishes camera_link -> depth/color/IR and
+    optical frames itself from the factory calibration, so none of those
+    frames are defined here. Depth FOV 91 x 66 deg, 50 mm baseline.
+  -->
+  <link name="camera_link"/>
+  <joint name="camera_joint" type="fixed">
+    <parent link="base_link"/>
+    <child link="camera_link"/>
+    <origin xyz="${camera_x} ${camera_y} ${camera_z}" rpy="0 ${camera_pitch} 0"/>
+  </joint>
 </robot>

Commit message: Localization and CPU: manual-pose scan matching, upright shadow filter, EventsExecutor
Real-vehicle driving on 2026-10-23 stalled in place and lost goals. Three
causes were found from the live topics and fixed:

- A web initial pose was 0.3 m / 15 deg off and AMCL settled there (match
  69 %, warnings every second). navigation_startup now scan-matches a manual
  or elevator prior within +-1 m / +-25 deg before AMCL verifies it
  (refine_pose; 7.8 % -> 74.7 % and 45 % -> 81 % on the vehicle, READY in
  9 s). The last READY pose is saved per map (~/.ros/amr_last_pose.json)
  and offered in the web UI as "이전 위치로 시작", applied only after the
  operator confirms it. The web UI sent the floor name with initial poses
  and the server rejected them; fixed.
- Beams grazing the 2020 upright edges return 0.36-0.50 m, outside the
  footprint, so the costmap carried lethal cells attached to the robot and
  DWB found no valid trajectory. scan_body_filter also clears each
  upright's shadow sector +-3 deg up to 0.7 m: near returns 32.6 -> 0 per
  scan, 1.3 % of valid beams removed, no "No valid trajectories" since.
- Python nodes overloaded the Jetson (load 12-15 on 6 cores);
  navigation_startup at 92 % starved its own TF listener and revoked READY
  13 times in 4 drives, and navigation_manager dropped the goal each time.
  Fixes: vehicle_status off by default; TF knots every 10 ms instead of a
  lookup per ray; raw particle cloud deserialized only while initializing;
  numpy scan validation; scoring only on new scan/pose pairs while READY;
  uncompensated score only when alignment fails; web_ui without deepcopy,
  numpy scan conversion and PNG encoding on request; EventsExecutor in the
  Python nodes (MessageInfo callbacks are unsupported by it, so /initialpose
  uses the fingerprint echo check). navigation_manager holds a goal at zero
  velocity for up to 5 s while a verified prior is re-verified, and an AMCL
  pose vs map->odom gap up to 1 m / 0.5 rad is a warning after READY
  (AMCL future-stamps its TF, so a correction blends briefly).

Measured after the changes: navigation_startup 92 % -> 22 %,
navigation_manager 38 % -> 3 %, web_ui 50-75 % -> 17 %, load 12-15 -> 4.8;
5 goals over two sessions reached with no stalls. IMU TF updated to the
v119 CAD position (0.097, 0, 0.021); the EKF fuses gyro Z only, so no
recalibration is needed.

Tests: package unit tests, elevator ROS tests and the integration runner
(manual, can_bridge, telemetry, ekf, localization, navigation_manager,
nav2_pipeline, web_ui, vehicle_status, navigation_startup 98, tim) pass on
the Jetson.

Co-Authored-By: Claude Fable 5.1 <noreply@anthropic.com>

File: src/amr_description/urdf/capstone_amr.urdf (robot description, URDF)
Before this commit: robot capstone_amr, 21 links, 20 joints
Joints:
- joint imu_joint: origin xyz=0.160 0.0035 0.016 rpy=0 0 0 -> xyz=0.097 0 0.021 rpy=0 0 0

File: src/amr_description/urdf/capstone_amr.urdf.xacro (robot description, xacro)
@@ -336,10 +336,12 @@
     <origin xyz="0 0 0" rpy="0 0 3.141592653589793"/>
   </joint>
-  <!-- LSM6DSV16X chip centre measured in CAD; axes match base_link. -->
+  <!-- LSM6DSV16X chip centre measured in CAD (v119 board position, 2026-10-23);
+       axes match base_link. The EKF fuses only gyro Z, so this offset does
+       not change the fused yaw rate. -->
   <link name="imu_link"/>
   <joint name="imu_joint" type="fixed">
     <parent link="base_link"/>
     <child link="imu_link"/>
-    <origin xyz="0.160 0.0035 0.016" rpy="0 0 0"/>
+    <origin xyz="0.097 0 0.021" rpy="0 0 0"/>
   </joint>
   <!--

File: src/amr_description/urdf/capstone_amr_physics.urdf (robot description, URDF)
Before this commit: robot capstone_amr, 21 links, 20 joints
Joints:
- joint imu_joint: origin xyz=0.160 0.0035 0.016 rpy=0 0 0 -> xyz=0.097 0 0.021 rpy=0 0 0

File: src/amr_description/urdf/capstone_amr_physics.urdf.xacro (robot description, xacro)
@@ -338,10 +338,12 @@
     <origin xyz="0 0 0" rpy="0 0 3.141592653589793"/>
   </joint>
-  <!-- LSM6DSV16X chip centre measured in CAD; axes match base_link. -->
+  <!-- LSM6DSV16X chip centre measured in CAD (v119 board position, 2026-10-23);
+       axes match base_link. The EKF fuses only gyro Z, so this offset does
+       not change the fused yaw rate. -->
   <link name="imu_link"/>
   <joint name="imu_joint" type="fixed">
     <parent link="base_link"/>
     <child link="imu_link"/>
-    <origin xyz="0.160 0.0035 0.016" rpy="0 0 0"/>
+    <origin xyz="0.097 0 0.021" rpy="0 0 0"/>
   </joint>
   <!--
