Commit message: WIP backup: depth camera integration and no-resume-approval work
Backup before fixing recovery clearing of depth obstacles; not yet
validated on the real vehicle.

- Gemini 2 depth camera: camera.launch.py, depth_layer in local and
  global costmaps, measured optical pitch 11.25 deg in URDF
- amr_depth_filter: drops depth obstacle points that do not persist
  for 3 frames (glossy-floor outliers); Release build by default
- Global costmap inflation_radius 1.6 -> 1.0 for straighter plans
- E-stop resume approval removal, elevator, web UI and remote bridge
  changes from the no-resume-approval branch

Co-Authored-By: Claude Opus 5.5 <noreply@anthropic.com>

File: src/amr_description/urdf/capstone_amr.urdf (robot description, URDF)
Before this commit: robot capstone_amr, 21 links, 20 joints
Joints:
- joint camera_joint: origin xyz=0.320488 0.025 0.061017 rpy=0 -0.20943951023931953 0 -> xyz=0.320488 0.025 0.061017 rpy=0 -0.19634954084936207 0

File: src/amr_description/urdf/capstone_amr.urdf.xacro (robot description, xacro)
@@ -46,4 +46,12 @@
   <xacro:property name="camera_z" value="0.061017"/>
   <xacro:property name="camera_pitch" value="${-12.0 * pi / 180.0}"/>
+  <!--
+    Depth optical axis as the ROS point cloud sees it: floor-plane fits on the
+    real vehicle (2026-10-25, three corridor spots, 0.34-1.82 m ahead) give
+    11.2-11.4 deg up, not the CAD 12 deg. With 12 deg the floor rose ~1.3 cm/m
+    and 2-3 m floor returns crossed the 5 cm marking height. The housing mesh
+    keeps the CAD pitch; only camera_joint uses the measured value.
+  -->
+  <xacro:property name="camera_optical_pitch" value="${-11.25 * pi / 180.0}"/>
   <!--
     18.0 kg total mass (set 2026-10-20 for v119; v28 measured 15.0 kg):
@@ -347,5 +355,5 @@
   <!--
     Orbbec Gemini 2 mount frame (+X along the optical axis, +Z up, pitched
-    12 deg up). OrbbecSDK_ROS2 publishes camera_link -> depth/color/IR and
+    11.25 deg up as measured; CAD 12 deg). OrbbecSDK_ROS2 publishes camera_link -> depth/color/IR and
     optical frames itself from the factory calibration, so none of those
     frames are defined here. Depth FOV 91 x 66 deg, 50 mm baseline.
@@ -355,5 +363,5 @@
     <parent link="base_link"/>
     <child link="camera_link"/>
-    <origin xyz="${camera_x} ${camera_y} ${camera_z}" rpy="0 ${camera_pitch} 0"/>
+    <origin xyz="${camera_x} ${camera_y} ${camera_z}" rpy="0 ${camera_optical_pitch} 0"/>
   </joint>
 </robot>
